File: board.kicad_pcb (KiCad board)
At the start: 2 copper layers, 100 x 65 mm, 62 parts, among them J1 JST_XH_Relays, J10 JST_XH_UART, J11 JST_HX_2, J12 JST-XH_LED_GND, J13 GS3, J14 GS3, J15 GS3, J16 JST_HX_2, J17 JST_HX_2, J18 JST_HX_2, J19 JST_HX_2, J2 2x40 2.5mm Header, J20 Conn_01x02, J21 Conn_01x02, J22 JST_XH_I2C, J23 JST_XH_I2C, J24 JST_XH_I2C, J25 JST_XH_I2C, J26 JST_XH_I2C, J27 JST_XH_I2C, J3 JST-XH_3, J4 JST-XH_3, J5 JST_HX_2, J6 Conn_02x04_Odd_Even, J7 JST-XH_3, J8 JST_HX_2, J9 JST-XH_3, Q1 IRLML6344TRPBF, Q2 IRLML6344TRPBF, Q3 IRLML6344TRPBF, Q4 IRLML6344TRPBF, Q5 IRLML6344TRPBF, SW1 SW_Push, SW2 SW_Push, SW3 SW_Push

Commit message: Syncing AISLER project with GitHub repository
Parts:
- C4: value 470uF -> 470u; footprint Capacitor_SMD:CP_Elec_10x10.5 -> Capacitor_SMD:CP_Elec_8x11.9
- moved G*** 1.36 mm to (156.3, 73.2)
- moved C4 0.60 mm to (135.0, 51.6)
Changed lines of the file:
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@@
   )
   (setup
-    (last_trace_width 2)
+    (last_trace_width 0.25)
     (user_trace_width 0.5)
     (user_trace_width 1)
@@
     (mod_text_size 1 1)
     (mod_text_width 0.15)
-    (pad_size 4.4 2.5)
+    (pad_size 4.15 1.9)
     (pad_drill 0)
     (pad_to_mask_clearance 0.2)
@@
     )
   )
+  (module Capacitor_SMD:CP_Elec_8x11.9 (layer F.Cu)
+    (at 135 51.6 180)
+    (descr "SMT capacitor, aluminium electrolytic, 8x11.9, Panasonic E12 ")
+    (tags "Capacitor Electrolytic")
+    (attr smd)
+    (fp_text reference C4 (at 0 -5.2 180) (layer F.SilkS)
+      (effects (font (size 1 1) (thickness 0.15)))
+    )
+    (fp_text value 470u (at 0 5.2 180) (layer F.Fab)
+      (effects (font (size 1 1) (thickness 0.15)))
+    )
+    (fp_circle (center 0 0) (end 4 0) (layer F.Fab) (width 0.1))
+    (fp_line (start 4.15 -4.15) (end 4.15 4.15) (layer F.Fab) (width 0.1))
+    (fp_line (start -3.15 -4.15) (end 4.15 -4.15) (layer F.Fab) (width 0.1))
+    (fp_line (start -3.15 4.15) (end 4.15 4.15) (layer F.Fab) (width 0.1))
+    (fp_line (start -4.15 -3.15) (end -4.15 3.15) (layer F.Fab) (width 0.1))
+    (fp_line (start -4.15 -3.15) (end -3.15 -4.15) (layer F.Fab) (width 0.1))
+    (fp_line (start -4.15 3.15) (end -3.15 4.15) (layer F.Fab) (width 0.1))
+    (fp_line (start -3.562278 -1.5) (end -2.762278 -1.5) (layer F.Fab) (width 0.1))
+    (fp_line (start -3.162278 -1.9) (end -3.162278 -1.1) (layer F.Fab) (width 0.1))
+    (fp_line (start 4.26 4.26) (end 4.26 1.21) (layer F.SilkS) (width 0.12))
+    (fp_line (start 4.26 -4.26) (end 4.26 -1.21) (layer F.SilkS) (width 0.12))
+    (fp_line (start -3.195563 -4.26) (end 4.26 -4.26) (layer F.SilkS) (width 0.12))
+    (fp_line (start -3.195563 4.26) (end 4.26 4.26) (layer F.SilkS) (width 0.12))
+    (fp_line (start -4.26 3.195563) (end -4.26 1.21) (layer F.SilkS) (width 0.12))
+    (fp_line (start -4.26 -3.195563) (end -4.26 -1.21) (layer F.SilkS) (width 0.12))
+    (fp_line (start -4.26 -3.195563) (end -3.195563 -4.26) (layer F.SilkS) (width 0.12))
+    (fp_line (start -4.26 3.195563) (end -3.195563 4.26) (layer F.SilkS) (width 0.12))
+    (fp_line (start -5.5 -2.21) (end -4.5 -2.21) (layer F.SilkS) (width 0.12))
+    (fp_line (start -5 -2.71) (end -5 -1.71) (layer F.SilkS) (width 0.12))
+    (fp_line (start 4.4 -4.4) (end 4.4 -1.2) (layer F.CrtYd) (width 0.05))
+    (fp_line (start 4.4 -1.2) (end 5.8 -1.2) (layer F.CrtYd) (width 0.05))
+    (fp_line (start 5.8 -1.2) (end 5.8 1.2) (layer F.CrtYd) (width 0.05))
+    (fp_line (start 5.8 1.2) (end 4.4 1.2) (layer F.CrtYd) (width 0.05))
+    (fp_line (start 4.4 1.2) (end 4.4 4.4) (layer F.CrtYd) (width 0.05))
+    (fp_line (start -3.25 4.4) (end 4.4 4.4) (layer F.CrtYd) (width 0.05))
+    (fp_line (start -3.25 -4.4) (end 4.4 -4.4) (layer F.CrtYd) (width 0.05))
+    (fp_line (start -4.4 3.25) (end -3.25 4.4) (layer F.CrtYd) (width 0.05))
+    (fp_line (start -4.4 -3.25) (end -3.25 -4.4) (layer F.CrtYd) (width 0.05))
+    (fp_line (start -4.4 -3.25) (end -4.4 -1.2) (layer F.CrtYd) (width 0.05))
+    (fp_line (start -4.4 1.2) (end -4.4 3.25) (layer F.CrtYd) (width 0.05))
+    (fp_line (start -4.4 -1.2) (end -5.8 -1.2) (layer F.CrtYd) (width 0.05))
+    (fp_line (start -5.8 -1.2) (end -5.8 1.2) (layer F.CrtYd) (width 0.05))
+    (fp_line (start -5.8 1.2) (end -4.4 1.2) (layer F.CrtYd) (width 0.05))
+    (fp_text user %R (at 0 0 180) (layer F.Fab)
+      (effects (font (size 1 1) (thickness 0.15)))
+    )
+    (pad 1 smd rect (at -3.475 0 180) (size 4.15 1.9) (layers F.Cu F.Paste F.Mask)
+      (net 42 +24V))
+    (pad 2 smd rect (at 3.475 0 180) (size 4.15 1.9) (layers F.Cu F.Paste F.Mask)
+      (net 2 GND) (zone_connect 2))
+    (model ${KISYS3DMOD}/Capacitor_SMD.3dshapes/CP_Elec_8x11.9.wrl
+      (at (xyz 0 0 0))
+      (scale (xyz 1 1 1))
+      (rotate (xyz 0 0 0))
+    )
+  )
   (module LED_SMD:LED_0603_1608Metric (layer F.Cu)
     (at 177.2 94.7 90)
@@
   )
   (module ressources:rocket3_Cu (layer B.Cu)
-    (at 154.94 73.2)
+    (at 156.3 73.2)
     (fp_text reference G*** (at 0 0) (layer B.SilkS) hide
       (effects (font (size 1.524 1.524) (thickness 0.3)) (justify mirror))
@@
       (xy -1.971615 1.454739) (xy -1.908759 1.469184)) (layer F.SilkS) (width 0.01))
   )
-  (module Capacitor_SMD:CP_Elec_10x10.5 (layer F.Cu)
-    (at 134.62 52.07 180)
-    (descr "SMT capacitor, aluminium electrolytic, 10x10, Vishay 1010 http://www.vishay.com/docs/28395/150crz.pdf")
-    (tags "Capacitor Electrolytic")
-    (attr smd)
-    (fp_text reference C4 (at 0 -6.3 180) (layer F.SilkS)
-      (effects (font (size 1 1) (thickness 0.15)))
-    )
-    (fp_text value 470uF (at 0 6.3 180) (layer F.Fab)
-      (effects (font (size 1 1) (thickness 0.15)))
-    )
-    (fp_circle (center 0 0) (end 5 0) (layer F.Fab) (width 0.1))
-    (fp_line (start 5.25 -5.25) (end 5.25 5.25) (layer F.Fab) (width 0.1))
-    (fp_line (start -4.25 -5.25) (end 5.25 -5.25) (layer F.Fab) (width 0.1))
-    (fp_line (start -4.25 5.25) (end 5.25 5.25) (layer F.Fab) (width 0.1))
-    (fp_line (start -5.25 -4.25) (end -5.25 4.25) (layer F.Fab) (width 0.1))
-    (fp_line (start -5.25 -4.25) (end -4.25 -5.25) (layer F.Fab) (width 0.1))
-    (fp_line (start -5.25 4.25) (end -4.25 5.25) (layer F.Fab) (width 0.1))
-    (fp_line (start -4.558325 -1.7) (end -3.558325 -1.7) (layer F.Fab) (width 0.1))
-    (fp_line (start -4.058325 -2.2) (end -4.058325 -1.2) (layer F.Fab) (width 0.1))
-    (fp_line (start 5.36 5.36) (end 5.36 1.51) (layer F.SilkS) (width 0.12))
-    (fp_line (start 5.36 -5.36) (end 5.36 -1.51) (layer F.SilkS) (width 0.12))
-    (fp_line (start -4.295563 -5.36) (end 5.36 -5.36) (layer F.SilkS) (width 0.12))
-    (fp_line (start -4.295563 5.36) (end 5.36 5.36) (layer F.SilkS) (width 0.12))
-    (fp_line (start -5.36 4.295563) (end -5.36 1.51) (layer F.SilkS) (width 0.12))
-    (fp_line (start -5.36 -4.295563) (end -5.36 -1.51) (layer F.SilkS) (width 0.12))
-    (fp_line (start -5.36 -4.295563) (end -4.295563 -5.36) (layer F.SilkS) (width 0.12))
-    (fp_line (start -5.36 4.295563) (end -4.295563 5.36) (layer F.SilkS) (width 0.12))
-    (fp_line (start -6.85 -2.76) (end -5.6 -2.76) (layer F.SilkS) (width 0.12))
-    (fp_line (start -6.225 -3.385) (end -6.225 -2.135) (layer F.SilkS) (width 0.12))
-    (fp_line (start 5.5 -5.5) (end 5.5 -1.5) (layer F.CrtYd) (width 0.05))
-    (fp_line (start 5.5 -1.5) (end 6.65 -1.5) (layer F.CrtYd) (width 0.05))
-    (fp_line (start 6.65 -1.5) (end 6.65 1.5) (layer F.CrtYd) (width 0.05))
-    (fp_line (start 6.65 1.5) (end 5.5 1.5) (layer F.CrtYd) (width 0.05))
-    (fp_line (start 5.5 1.5) (end 5.5 5.5) (layer F.CrtYd) (width 0.05))
-    (fp_line (start -4.35 5.5) (end 5.5 5.5) (layer F.CrtYd) (width 0.05))
-    (fp_line (start -4.35 -5.5) (end 5.5 -5.5) (layer F.CrtYd) (width 0.05))
-    (fp_line (start -5.5 4.35) (end -4.35 5.5) (layer F.CrtYd) (width 0.05))
-    (fp_line (start -5.5 -4.35) (end -4.35 -5.5) (layer F.CrtYd) (width 0.05))
-    (fp_line (start -5.5 -4.35) (end -5.5 -1.5) (layer F.CrtYd) (width 0.05))
-    (fp_line (start -5.5 1.5) (end -5.5 4.35) (layer F.CrtYd) (width 0.05))
-    (fp_line (start -5.5 -1.5) (end -6.65 -1.5) (layer F.CrtYd) (width 0.05))
-    (fp_line (start -6.65 -1.5) (end -6.65 1.5) (layer F.CrtYd) (width 0.05))
-    (fp_line (start -6.65 1.5) (end -5.5 1.5) (layer F.CrtYd) (width 0.05))
-    (fp_text user %R (at 0 0 180) (layer F.Fab)
-      (effects (font (size 1 1) (thickness 0.15)))
-    )
-    (pad 1 smd rect (at -4.2 0 180) (size 4.4 2.5) (layers F.Cu F.Paste F.Mask)
-      (net 42 +24V))
-    (pad 2 smd rect (at 4.2 0 180) (size 4.4 2.5) (layers F.Cu F.Paste F.Mask)
-      (net 2 GND) (zone_connect 2))
-    (model ${KISYS3DMOD}/Capacitor_SMD.3dshapes/CP_Elec_10x10.5.wrl
-      (at (xyz 0 0 0))
-      (scale (xyz 1 1 1))
-      (rotate (xyz 0 0 0))
-    )
-  )
   (dimension 83 (width 0.25) (layer Eco2.User)
     (gr_text "83.000 mm" (at 155 121) (layer Eco2.User)
@@
     (effects (font (size 1 1) (thickness 0.2)))
   )
-  (gr_text "AstroPlant Mk06\nProto - VFR" (at 134.62 72.39 90) (layer F.SilkS)
+  (gr_text "AstroPlant Mk06\nProto - VFR" (at 134.9 70.7 90) (layer F.SilkS)
     (effects (font (size 1 1) (thickness 0.2)) (justify left))
   )
@@
   (segment (start 125.8 57) (end 124.775 55.975) (width 2) (layer F.Cu) (net 41))
   (via (at 143.3 52.3) (size 2.1) (drill 0.6) (layers F.Cu B.Cu) (net 42))
+  (segment (start 138.475 51.6) (end 142.6 51.6) (width 2) (layer F.Cu) (net 42))
+  (segment (start 142.6 51.6) (end 143.3 52.3) (width 2) (layer F.Cu) (net 42))
   (via (at 151.4 52.3) (size 2.1) (drill 0.6) (layers F.Cu B.Cu) (net 42))
   (segment (start 143.3 52.3) (end 151.4 52.3) (width 2) (layer B.Cu) (net 42))
@@
   (via (at 174.3 52.3) (size 2.1) (drill 0.6) (layers F.Cu B.Cu) (net 42))
   (segment (start 162.6 52.3) (end 174.3 52.3) (width 2) (layer B.Cu) (net 42))
+  (segment (start 137.2 50.325) (end 138.475 51.6) (width 2) (layer F.Cu) (net 42))
+  (segment (start 137.2 41.4) (end 137.2 50.325) (width 2) (layer F.Cu) (net 42))
   (segment (start 151.4 53.784924) (end 151.4 55.09999) (width 2) (layer F.Cu) (net 42))
   (segment (start 151.4 52.3) (end 151.4 53.784924) (width 2) (layer F.Cu) (net 42))
@@
   (segment (start 162.6 52.3) (end 162.6 53.784924) (width 2) (layer F.Cu) (net 42))
   (segment (start 174.3 52.3) (end 174.3 54.89999) (width 2) (layer F.Cu) (net 42))
-  (segment (start 137.2 50.45) (end 138.82 52.07) (width 2) (layer F.Cu) (net 42))
-  (segment (start 137.2 41.4) (end 137.2 50.45) (width 2) (layer F.Cu) (net 42))
-  (segment (start 139.05 52.3) (end 138.82 52.07) (width 2) (layer F.Cu) (net 42))
-  (segment (start 143.3 52.3) (end 139.05 52.3) (width 2) (layer F.Cu) (net 42))
   (zone (net 2) (net_name GND) (layer F.Cu) (hatch edge 0.508)
     (connect_pads (clearance 0.508))
